File: kicad/valentines-heart-punk-r1.2-rotated.kicad_pcb (KiCad board)
At the start: 2 copper layers, 49.5 x 49.5 mm, 28 parts, among them SW1 SW_Push, U1 ATtiny25-20S

Commit message: Updating layout
Parts:
- BT1: value BatteryHolder_Keystone_1060_1x2032 -> Battery_Cell
Connections:
- BT1 pad 1: (no net) -> +3.3V
- BT1 pad 2: (no net) -> GND
- C1 pad 1: +3V3 -> +3.3V
- U1 pad 8: +3V3 -> +3.3V
Routing:
- net +3V3: track 19.1 -> 0.00 mm, vias 1 -> 0
- net +3.3V: track 0.00 -> 19.1 mm, vias 0 -> 1
